Commit message: minor updates

File: urdf/c5.urdf.xacro (robot description, xacro)
@@ -16,7 +16,4 @@
                 <mesh filename="file:///$(find leica_gazebo_simulation)/meshes/scanstation_c5.dae" scale="0.001 0.001 0.001"/>
             </geometry>
-            <!-- <material name="Red">
-                <color rgba="0.7 0.7 0.7 0.7"/>
-            </material> -->
         </visual>
         <collision>

File: urdf/sensor.urdf.xacro (robot description, xacro)
@@ -31,18 +31,17 @@
             <pose>0 0 0 0 0 0</pose>
             <visualize>true</visualize>
-            <update_rate>40</update_rate>            <!--105-->
+            <update_rate>40</update_rate>
             <ray>
                 <scan>
                     <horizontal>
-                        <samples>1</samples>
-                        <resolution>1024</resolution>                        <!--1024-->
-                        <min_angle>-1.4</min_angle>    <!---1.57-->
-                        <max_angle>1.4</max_angle>     <!--1.57-->
+                        <samples>512</samples>
+                        <resolution>1</resolution>
+                        <min_angle>-1.04</min_angle> <!-- Be sure the angle between min and max angle is > 1.5708 -->
+                        <max_angle>0.8</max_angle>
                     </horizontal>
                 </scan>
                 <range>
-                    <min>0.35</min>
+                    <min>0.15</min>
                     <max>8.0</max>
-                    <max>50.0</max>
                     <resolution>0.004</resolution>
                 </range>
@@ -50,5 +49,5 @@
                     <type>gaussian</type>
                     <mean>0.0</mean>
-                    <stddev>0.002</stddev>
+                    <stddev>0.0</stddev>
                 </noise>
             </ray>
@@ -56,5 +55,4 @@
                 <topicName>/c5/simulator/scan</topicName>
                 <frameName>sensor_link</frameName>
-                <!--update_rate>40</update_rate-->
             </plugin>
         </sensor>
